File: LV_FINAL.kicad_sch (KiCad schematic)
At the start: 0 parts

Commit message: Add files via upload
Other:
- sheet SHUTDOWN_CIRCUIT ports: added HV_PRECHARGE, LV+_AMS1, LV+_AMS2; removed BSPD_OUT, IMD_OUT, LVMS_OUT
