File: precharge.kicad_sch (KiCad schematic)
At the start: 28 parts, among them Q5 BC107, U10 74HC7014, U11 74LS08, U12 74LS21, U13 74LVC2G04, U14 74LVC1G175, U15 74LVC1G175, U16 74LVC1G175, U17 4060, U18 74LVC1G175

Commit message: update
Connections:
- net PCR+ renamed HIGHVOLTAGE_PR
Changed lines of the file:
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@@
+		)
+	)
+	(hierarchical_label "HIGHVOLTAGE_PR"
+		(shape input)
+		(at 92.71 55.88 0)
+		(fields_autoplaced yes)
+		(effects
+			(font
+				(size 1.27 1.27)
+			)
+			(justify left)
 		)
 	)
