File: untitled.kicad_sch (KiCad schematic)
At the start: 14 parts, among them SW10 SW_SPST, SW6 SW_SPST, SW7 SW_SPST, SW8 SW_SPST, SW9 SW_SPST, sw1 SW_SPST, sw11 SW_SPST, sw2 SW_SPST, sw3 SW_SPST, sw4 SW_SPST, sw5 SW_SPST

Commit message: update
Other:
- sheet AMS ports: added LOWVOLTAGE_PIN1, LOWVOLTAGE_PIN2; removed none
- sheet Precharge ports: added HIGHVOLTAGE_PR; removed none
Changed lines of the file:
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@@
+	(wire
+		(pts
+			(xy 176.53 185.42) (xy 182.88 185.42)
+		)
+		(stroke
+			(width 0)
+			(type default)
+		)
+	)
 	(wire
 		(pts
@@
 	(wire
 		(pts
-			(xy 238.76 190.5) (xy 243.84 190.5)
+			(xy 224.79 189.23) (xy 229.87 189.23)
 		)
 		(stroke
@@
 	(wire
 		(pts
+			(xy 176.53 187.96) (xy 182.88 187.96)
+		)
+		(stroke
+			(width 0)
+			(type default)
+		)
+	)
+	(wire
+		(pts
 			(xy 228.6 55.88) (xy 217.17 55.88)
 		)
@@
 	(wire
 		(pts
+			(xy 224.79 191.77) (xy 229.87 191.77)
+		)
+		(stroke
+			(width 0)
+			(type default)
+		)
+	)
+	(wire
+		(pts
 			(xy 87.63 118.11) (xy 87.63 121.92)
 		)
@@
 	(wire
 		(pts
-			(xy 236.22 187.96) (xy 243.84 187.96)
+			(xy 222.25 186.69) (xy 229.87 186.69)
 		)
 		(stroke
@@
 		)
 	)
+	(hierarchical_label "LV+_AMS1"
+		(shape input)
+		(at 176.53 185.42 180)
+		(fields_autoplaced yes)
+		(effects
+			(font
+				(size 1.27 1.27)
+				(bold yes)
+			)
+			(justify right)
+		)
+	)
 	(hierarchical_label "LV+_BSPD"
 		(shape input)
@@
 	(hierarchical_label "LV+_PRECHARGE"
 		(shape input)
-		(at 236.22 187.96 180)
+		(at 222.25 186.69 180)
 		(fields_autoplaced yes)
 		(effects
@@
 		)
 	)
+	(hierarchical_label "LV+_AMS2"
+		(shape input)
+		(at 176.53 187.96 180)
+		(fields_autoplaced yes)
+		(effects
+			(font
+				(size 1.27 1.27)
+				(bold yes)
+			)
+			(justify right)
+		)
+	)
 	(hierarchical_label "HV-_IMD"
 		(shape input)
@@
 	(hierarchical_label "LV_GND_PRECHARGE"
 		(shape input)
-		(at 238.76 190.5 180)
+		(at 224.79 189.23 180)
 		(fields_autoplaced yes)
 		(effects
@@
 			)
 			(justify left)
+		)
+	)
+	(hierarchical_label "HV_PRECHARGE"
+		(shape input)
+		(at 224.79 191.77 180)
+		(fields_autoplaced yes)
+		(effects
+			(font
+				(size 1.27 1.27)
+				(bold yes)
+			)
+			(justify right)
 		)
 	)
@@
 		(fields_autoplaced yes)
 		(stroke
-			(width 0.1524)
+			(width 0.5)
 			(type solid)
 		)
@@
 	)
 	(sheet
-		(at 243.84 181.61)
+		(at 229.87 180.34)
 		(size 17.78 34.29)
 		(fields_autoplaced yes)
 		(stroke
-			(width 0.1524)
+			(width 0.5)
 			(type solid)
 		)
@@
 		)
 		(property "Sheetname" "Precharge"
-			(at 243.84 180.5334 0)
+			(at 229.87 179.2634 0)
 			(effects
 				(font
@@
 		)
 		(property "Sheetfile" "precharge.kicad_sch"
-			(at 243.84 216.4846 0)
+			(at 229.87 215.2146 0)
 			(effects
 				(font
@@
 		)
 		(pin "LV+" input
-			(at 243.84 187.96 180)
+			(at 229.87 186.69 180)
 			(effects
 				(font
@@
 		)
 		(pin "LV_GND" input
-			(at 243.84 190.5 180)
+			(at 229.87 189.23 180)
+			(effects
+				(font
+					(size 1.27 1.27)
+				)
+				(justify left)
+			)
+		)
+		(pin "HIGHVOLTAGE_PR" input
+			(at 229.87 191.77 180)
 			(effects
 				(font
@@
 		(fields_autoplaced yes)
 		(stroke
-			(width 0.1524)
+			(width 0.5)
 			(type solid)
 		)
@@
 	)
 	(sheet
-		(at 194.31 180.34)
-		(size 17.78 35.56)
-		(fields_autoplaced yes)
-		(stroke
-			(width 0.1524)
+		(at 182.88 180.34)
+		(size 19.05 35.56)
+		(fields_autoplaced yes)
+		(stroke
+			(width 0.5)
 			(type solid)
 		)
@@
 		)
 		(property "Sheetname" "AMS"
-			(at 194.31 179.2634 0)
+			(at 182.88 179.2634 0)
 			(effects
 				(font
@@
 		)
 		(property "Sheetfile" "AMS.kicad_sch"
-			(at 194.31 216.4846 0)
+			(at 182.88 216.4846 0)
 			(effects
 				(font
@@
 			)
 		)
+		(pin "LOWVOLTAGE_PIN2" input
+			(at 182.88 185.42 180)
+			(effects
+				(font
+					(size 1.27 1.27)
+				)
+				(justify left)
+			)
+		)
+		(pin "LOWVOLTAGE_PIN1" input
+			(at 182.88 187.96 180)
+			(effects
+				(font
+					(size 1.27 1.27)
+				)
+				(justify left)
+			)
+		)
